Commit message: add linker hand

File: openarm_description/urdf/openarm_with_linker_hand.urdf (robot description, URDF)
Before this commit: robot openarm, 30 links, 29 joints
Links:
- added link base_link
Joints:
- added joint world_to_pedestal: type fixed, parent world, child base_link, origin xyz=0.0 0.0 0.0 rpy=0.0 0.0 0.0

Commit message: update

File: openarm_description/urdf/openarm_with_linker_hand.urdf (robot description, URDF)
Before this commit: robot openarm, 31 links, 30 joints
Links:
- added link openarm_right_hand, mass 0.35; collision mesh filename=package://openarm_description/meshes/ee/openarm_hand/collis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 scale=0.001 0.001 0.001; visual mesh filename=package://openarm_description/meshes/ee/openarm_hand/visual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 scale=0.001 0.001 0.001
- added link openarm_right_hand_tcp
- added link openarm_right_left_finger, mass 0.03602545343277134; collision mesh filename=package://openarm_description/meshes/ee/openarm_hand/collis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 scale=0.001 0.001 0.001; visual mesh filename=package://openarm_description/meshes/ee/openarm_hand/visual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 scale=0.001 0.001 0.001
- added link openarm_right_right_finger, mass 0.03602545343277134; collision mesh filename=package://openarm_description/meshes/ee/openarm_hand/collis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 scale=0.001 -0.001 0.001; visual mesh filename=package://openarm_description/meshes/ee/openarm_hand/visual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 scale=0.001 -0.001 0.001
Joints:
- added joint openarm_right_finger_joint1: type prismatic, parent openarm_right_hand, child openarm_right_right_finger, origin xyz=0 -0.006 0.015 rpy=0 0 0, axis 0 -1 0, limit lower=0.0 upper=0.044 effort=333 velocity=10.0
- added joint openarm_right_finger_joint2: type prismatic, parent openarm_right_hand, child openarm_right_left_finger, origin xyz=0 0.006 0.015 rpy=0 0 0, axis 0 1 0, limit lower=0.0 upper=0.044 effort=333 velocity=10.0, mimic joint=openarm_right_finger_joint1
- added joint openarm_right_hand_tcp_joint: type fixed, parent openarm_right_hand, child openarm_right_hand_tcp, origin xyz=0 -0.0 0.08 rpy=0 0 0
- added joint right_openarm_hand_joint: type fixed, parent openarm_right_link7, child openarm_right_hand, origin xyz=0 -0.0 0.1001 rpy=0 0 0
